Commit message: URDF update and arxiv preprint

File: src/hand_rviz/urdf/hand_urdf.urdf (robot description, URDF)
Before this commit: robot hand_rviz/urdf, 22 links, 21 joints
Links:
- added link i_tip_link, mass 9.6341391738565E-05; collision mesh filename=package://hand_rviz/urdf/meshes/i_tip_link.STL; visual mesh filename=package://hand_rviz/urdf/meshes/i_tip_link.STL
- added link m_tip_link, mass 9.63413917385605E-05; collision mesh filename=package://hand_rviz/urdf/meshes/m_tip_link.STL; visual mesh filename=package://hand_rviz/urdf/meshes/m_tip_link.STL
- added link p_tip_link, mass 9.63413917385593E-05; collision mesh filename=package://hand_rviz/urdf/meshes/p_tip_link.STL; visual mesh filename=package://hand_rviz/urdf/meshes/p_tip_link.STL
- added link r_tip_link, mass 9.63413917385707E-05; collision mesh filename=package://hand_rviz/urdf/meshes/r_tip_link.STL; visual mesh filename=package://hand_rviz/urdf/meshes/r_tip_link.STL
- added link t_tip_link, mass 9.63413917384506E-05; collision mesh filename=package://hand_rviz/urdf/meshes/t_tip_link.STL; visual mesh filename=package://hand_rviz/urdf/meshes/t_tip_link.STL
- link hand_base_link: mass 1.3833 -> 1.38812640347778
- link idf_link: mass 0.00213606646468501 -> 0.00213606646468497
- link ima_link: mass 0.003771 -> 0.00377097433248701
- link imf_link: mass 0.00350627784467482 -> 0.0035062778446748
- link mdf_link: mass 0.00213606647535569 -> 0.00213606647535568
- link mmf_link: mass 0.00350627793815242 -> 0.0035062779381524
- link mpf_link: mass 0.00108838501206663 -> 0.00108838501206664
- link pdf_link: mass 0.00213606649935728 -> 0.00213606649935726
- link pma_link: mass 0 -> 0.00377097300672915
- link pmf_link: mass 0.0035062779898751 -> 0.00350627798987508
- link rdf_link: mass 0.00213606648739499 -> 0.002136066487395
- link rmf_link: mass 0.00350627800305114 -> 0.00350627800305113
- link rpf_link: mass 0.00108838501206663 -> 0.00108838501206664
- link tma_link: mass 0.00313620364525098 -> 0.00320272686969075
- link tmf_link: mass 0.000948811114997918 -> 0.000948811114997913
Joints:
- added joint i_tip: type fixed, parent idf_link, child i_tip_link, origin xyz=0.0091323 0 0 rpy=0 0 0, axis 0 0 0
- added joint m_tip: type fixed, parent mdf_link, child m_tip_link, origin xyz=0.0091323 0 0 rpy=0 0 0, axis 0 0 0
- added joint p_tip: type fixed, parent pdf_link, child p_tip_link, origin xyz=0.00913233682828257 0 0 rpy=0 0 0, axis 0 0 0
- added joint r_tip: type fixed, parent rdf_link, child r_tip_link, origin xyz=0.00913233682828257 0 0 rpy=0 0 0, axis 0 0 0
- added joint t_tip: type fixed, parent tdf_link, child t_tip_link, origin xyz=0.012137 0 0 rpy=0 0 0, axis 0 0 0
- joint idf_joint: limit lower=-1.57 upper=1.57 effort=0 velocity=0 -> lower=0 upper=1.25 effort=0 velocity=0; origin xyz=0.02618 0 0 rpy=0 0 0.397620554199505 -> xyz=0.02618 0 0 rpy=0 0 0.39762
- joint ima_joint: axis 0 0 -1 -> 0 0 1; origin xyz=-0.030085 -0.038 0.11024 rpy=1.5708 -1.4573 -3.1416 -> xyz=-0.030085 -0.0405 0.11024 rpy=-1.5708 -1.4573 -3.1416
- joint imf_joint: origin xyz=0.017 0.0045 -0.001625 rpy=1.5708 0 0 -> xyz=0.017 0 -0.000875 rpy=-1.5708 0 0
- joint ipf_joint: origin xyz=0.031 0 0.00244999999999999 rpy=0 0 1.17317577259539 -> xyz=0.031 0 0 rpy=0 0 1.1732
- joint mdf_joint: limit lower=-1.57 upper=1.57 effort=0 velocity=0 -> lower=0 upper=1.25 effort=0 velocity=0; origin xyz=0.02618 0 0 rpy=0 0 0.397620554199505 -> xyz=0.02618 0 0 rpy=0 0 0.39762
- joint mma_joint: axis 0 0 -1 -> 0 0 1; origin xyz=-0.010267 -0.038 0.12046 rpy=1.5708 -1.5272 -3.1416 -> xyz=-0.010267 -0.0405 0.12046 rpy=-1.5708 -1.5272 -3.1416
- joint mmf_joint: origin xyz=0.017 0.0045 -0.001625 rpy=1.5708 0 0 -> xyz=0.017 0 -0.000875 rpy=-1.5708 0 0
- joint mpf_joint: origin xyz=0.0309999999999998 0 0.00245 rpy=0 0 1.17317577259539 -> xyz=0.031 0 0 rpy=0 0 1.1732
- joint pdf_joint: limit lower=-1.57 upper=1.57 effort=0 velocity=0 -> lower=0 upper=1.25 effort=0 velocity=0
- joint pma_joint: axis 0 0 -1 -> 0 0 1; origin xyz=0.030085 -0.038 0.11024 rpy=-1.5708 -1.4573 0 -> xyz=0.030085 -0.0405 0.11024 rpy=1.5708 -1.4573 0
- joint pmf_joint: origin xyz=0.017 0.0045 -0.001625 rpy=1.5707963267949 0 0 -> xyz=0.017 0 -0.000875 rpy=-1.5707963267949 0 0
- joint ppf_joint: origin xyz=0.0309999999999999 0 0.00245 rpy=0 0 1.17317577259539 -> xyz=0.031 0 0 rpy=0 0 1.17317577259539
- joint rdf_joint: limit lower=-1.57 upper=1.57 effort=0 velocity=0 -> lower=0 upper=1.25 effort=0 velocity=0
- joint rma_joint: axis 0 0 -1 -> 0 0 1; origin xyz=0.010267 -0.038 0.12046 rpy=-1.5708 -1.5272 0 -> xyz=0.010267 -0.0405 0.12046 rpy=1.5708 -1.5272 0
- joint rmf_joint: origin xyz=0.017 0.00450000000000001 -0.001625 rpy=1.5707963267949 0 0 -> xyz=0.017 0 -0.000875 rpy=-1.5708 0 0
- joint rpf_joint: origin xyz=0.031 0 0.00245 rpy=0 0 1.17317577259539 -> xyz=0.031 0 0 rpy=0 0 1.17317577259539
- joint tca_joint: origin xyz=-0.024 0.014785 0.0072407 rpy=2.8032 -1.0121 1.9642 -> xyz=-0.024 0.01695 0.011491 rpy=2.8032 -1.0121 1.9642
- joint tcf_joint: origin xyz=-0.03245 -0.0217 0.055 rpy=0 0 0 -> xyz=-0.03245 -0.0217 0.0495 rpy=0 0 0
- joint tdf_joint: limit lower=-1.57 upper=1.57 effort=0 velocity=0 -> lower=0 upper=1.25 effort=0 velocity=0; origin xyz=0.025 0 0 rpy=0 0 0.128195437634862 -> xyz=0.025 0 0 rpy=0 0 0.1282
- joint tma_joint: origin xyz=0.025 0.00304267643461039 0.0026 rpy=-1.5707963267949 0.27478795531439 0 -> xyz=0.025 -0.0014573 0.0001 rpy=-1.5708 0.27479 0
- joint tmf_joint: origin xyz=0.0199999999999999 0.00199999999999999 -0.003 rpy=1.5707963267949 -0.346793637861002 0 -> xyz=0.02 0 0.0015 rpy=1.5708 -0.34679 0

File: src/hand_rviz/urdf/hand_urdf_cf.urdf (robot description, URDF)
Before this commit: robot hand_rviz/urdf, 22 links, 21 joints
Links:
- added link i_tip_link, mass 9.6341391738565E-05; collision mesh filename=package://hand_rviz/urdf/meshes/i_tip_link.STL; visual mesh filename=package://hand_rviz/urdf/meshes/i_tip_link.STL
- added link m_tip_link, mass 9.63413917385605E-05; collision mesh filename=package://hand_rviz/urdf/meshes/m_tip_link.STL; visual mesh filename=package://hand_rviz/urdf/meshes/m_tip_link.STL
- added link p_tip_link, mass 9.63413917385593E-05; collision mesh filename=package://hand_rviz/urdf/meshes/p_tip_link.STL; visual mesh filename=package://hand_rviz/urdf/meshes/p_tip_link.STL
- added link r_tip_link, mass 9.63413917385707E-05; collision mesh filename=package://hand_rviz/urdf/meshes/r_tip_link.STL; visual mesh filename=package://hand_rviz/urdf/meshes/r_tip_link.STL
- added link t_tip_link, mass 9.63413917384506E-05; collision mesh filename=package://hand_rviz/urdf/meshes/t_tip_link.STL; visual mesh filename=package://hand_rviz/urdf/meshes/t_tip_link.STL
- link hand_base_link: mass 1.3833 -> 1.38812640347778; geometry collision mesh filename=package://hand_rviz/urdf/meshes/hand_base_link.STL; visual mesh filename=package://hand_rviz/urdf/meshes/hand_base_link.STL
- link idf_link: mass 0.00213606646468501 -> 0.00213606646468497; geometry collision mesh filename=package://hand_rviz/urdf/meshes/idf_link.STL; visual mesh filename=package://hand_rviz/urdf/meshes/idf_link.STL
- link ima_link: mass 0.003771 -> 0.00377097433248701; geometry collision mesh filename=package://hand_rviz/urdf/meshes/ima_link.STL; visual mesh filename=package://hand_rviz/urdf/meshes/ima_link.STL
- link imf_link: mass 0.00350627784467482 -> 0.0035062778446748; geometry collision mesh filename=package://hand_rviz/urdf/meshes/imf_link.STL; visual mesh filename=package://hand_rviz/urdf/meshes/imf_link.STL
- link ipf_link: geometry collision mesh filename=package://hand_rviz/urdf/meshes/ipf_link.STL; visual mesh filename=package://hand_rviz/urdf/meshes/ipf_link.STL
- link mdf_link: mass 0.00213606647535569 -> 0.00213606647535568; geometry collision mesh filename=package://hand_rviz/urdf/meshes/mdf_link.STL; visual mesh filename=package://hand_rviz/urdf/meshes/mdf_link.STL
- link mma_link: geometry collision mesh filename=package://hand_rviz/urdf/meshes/mma_link.STL; visual mesh filename=package://hand_rviz/urdf/meshes/mma_link.STL
- link mmf_link: mass 0.00350627793815242 -> 0.0035062779381524; geometry collision mesh filename=package://hand_rviz/urdf/meshes/mmf_link.STL; visual mesh filename=package://hand_rviz/urdf/meshes/mmf_link.STL
- link mpf_link: mass 0.00108838501206663 -> 0.00108838501206664; geometry collision mesh filename=package://hand_rviz/urdf/meshes/mpf_link.STL; visual mesh filename=package://hand_rviz/urdf/meshes/mpf_link.STL
- link pdf_link: mass 0.00213606649935728 -> 0.00213606649935726; geometry collision mesh filename=package://hand_rviz/urdf/meshes/pdf_link.STL; visual mesh filename=package://hand_rviz/urdf/meshes/pdf_link.STL
- link pma_link: mass 0 -> 0.00377097300672915; geometry collision mesh filename=package://hand_rviz/urdf/meshes/pma_link.STL; visual mesh filename=package://hand_rviz/urdf/meshes/pma_link.STL
- link pmf_link: mass 0.0035062779898751 -> 0.00350627798987508; geometry collision mesh filename=package://hand_rviz/urdf/meshes/pmf_link.STL; visual mesh filename=package://hand_rviz/urdf/meshes/pmf_link.STL
- link ppf_link: geometry collision mesh filename=package://hand_rviz/urdf/meshes/ppf_link.STL; visual mesh filename=package://hand_rviz/urdf/meshes/ppf_link.STL
- link rdf_link: mass 0.00213606648739499 -> 0.002136066487395; geometry collision mesh filename=package://hand_rviz/urdf/meshes/rdf_link.STL; visual mesh filename=package://hand_rviz/urdf/meshes/rdf_link.STL
- link rma_link: geometry collision mesh filename=package://hand_rviz/urdf/meshes/rma_link.STL; visual mesh filename=package://hand_rviz/urdf/meshes/rma_link.STL
- link rmf_link: mass 0.00350627800305114 -> 0.00350627800305113; geometry collision mesh filename=package://hand_rviz/urdf/meshes/rmf_link.STL; visual mesh filename=package://hand_rviz/urdf/meshes/rmf_link.STL
- link rpf_link: mass 0.00108838501206663 -> 0.00108838501206664; geometry collision mesh filename=package://hand_rviz/urdf/meshes/rpf_link.STL; visual mesh filename=package://hand_rviz/urdf/meshes/rpf_link.STL
- link tca_link: geometry collision mesh filename=package://hand_rviz/urdf/meshes/tca_link.STL; visual mesh filename=package://hand_rviz/urdf/meshes/tca_link.STL
- link tcf_link: geometry collision mesh filename=package://hand_rviz/urdf/meshes/tcf_link.STL; visual mesh filename=package://hand_rviz/urdf/meshes/tcf_link.STL
- link tdf_link: geometry collision mesh filename=package://hand_rviz/urdf/meshes/tdf_link.STL; visual mesh filename=package://hand_rviz/urdf/meshes/tdf_link.STL
- link tma_link: mass 0.00313620364525098 -> 0.00320272686969075; geometry collision mesh filename=package://hand_rviz/urdf/meshes/tma_link.STL; visual mesh filename=package://hand_rviz/urdf/meshes/tma_link.STL
- link tmf_link: mass 0.000948811114997918 -> 0.000948811114997913; geometry collision mesh filename=package://hand_rviz/urdf/meshes/tmf_link.STL; visual mesh filename=package://hand_rviz/urdf/meshes/tmf_link.STL
Joints:
- added joint i_tip: type fixed, parent idf_link, child i_tip_link, origin xyz=0.0091323 0 0 rpy=0 0 0, axis 0 0 0
- added joint m_tip: type fixed, parent mdf_link, child m_tip_link, origin xyz=0.0091323 0 0 rpy=0 0 0, axis 0 0 0
- added joint p_tip: type fixed, parent pdf_link, child p_tip_link, origin xyz=0.00913233682828257 0 0 rpy=0 0 0, axis 0 0 0
- added joint r_tip: type fixed, parent rdf_link, child r_tip_link, origin xyz=0.00913233682828257 0 0 rpy=0 0 0, axis 0 0 0
- added joint t_tip: type fixed, parent tdf_link, child t_tip_link, origin xyz=0.012137 0 0 rpy=0 0 0, axis 0 0 0
- joint idf_joint: limit lower=-1.57 upper=1.57 effort=0 velocity=0 -> lower=0 upper=1.25 effort=0 velocity=0; origin xyz=0.02618 0 0 rpy=0 0 0.397620554199505 -> xyz=0.02618 0 0 rpy=0 0 0.39762
- joint ima_joint: axis 0 0 -1 -> 0 0 1; origin xyz=-0.030085 -0.038 0.11024 rpy=1.5708 -1.4573 -3.1416 -> xyz=-0.030085 -0.0405 0.11024 rpy=-1.5708 -1.4573 -3.1416
- joint imf_joint: origin xyz=0.017 0.0045 -0.001625 rpy=1.5708 0 0 -> xyz=0.017 0 -0.000875 rpy=-1.5708 0 0
- joint ipf_joint: origin xyz=0.031 0 0.00244999999999999 rpy=0 0 1.17317577259539 -> xyz=0.031 0 0 rpy=0 0 1.1732
- joint mdf_joint: limit lower=-1.57 upper=1.57 effort=0 velocity=0 -> lower=0 upper=1.25 effort=0 velocity=0; origin xyz=0.02618 0 0 rpy=0 0 0.397620554199505 -> xyz=0.02618 0 0 rpy=0 0 0.39762
- joint mma_joint: axis 0 0 -1 -> 0 0 1; origin xyz=-0.010267 -0.038 0.12046 rpy=1.5708 -1.5272 -3.1416 -> xyz=-0.010267 -0.0405 0.12046 rpy=-1.5708 -1.5272 -3.1416
- joint mmf_joint: origin xyz=0.017 0.0045 -0.001625 rpy=1.5708 0 0 -> xyz=0.017 0 -0.000875 rpy=-1.5708 0 0
- joint mpf_joint: origin xyz=0.0309999999999998 0 0.00245 rpy=0 0 1.17317577259539 -> xyz=0.031 0 0 rpy=0 0 1.1732
- joint pdf_joint: limit lower=-1.57 upper=1.57 effort=0 velocity=0 -> lower=0 upper=1.25 effort=0 velocity=0
- joint pma_joint: axis 0 0 -1 -> 0 0 1; origin xyz=0.030085 -0.038 0.11024 rpy=-1.5708 -1.4573 0 -> xyz=0.030085 -0.0405 0.11024 rpy=1.5708 -1.4573 0
- joint pmf_joint: origin xyz=0.017 0.0045 -0.001625 rpy=1.5707963267949 0 0 -> xyz=0.017 0 -0.000875 rpy=-1.5707963267949 0 0
- joint ppf_joint: origin xyz=0.0309999999999999 0 0.00245 rpy=0 0 1.17317577259539 -> xyz=0.031 0 0 rpy=0 0 1.17317577259539
- joint rdf_joint: limit lower=-1.57 upper=1.57 effort=0 velocity=0 -> lower=0 upper=1.25 effort=0 velocity=0
- joint rma_joint: axis 0 0 -1 -> 0 0 1; origin xyz=0.010267 -0.038 0.12046 rpy=-1.5708 -1.5272 0 -> xyz=0.010267 -0.0405 0.12046 rpy=1.5708 -1.5272 0
- joint rmf_joint: origin xyz=0.017 0.00450000000000001 -0.001625 rpy=1.5707963267949 0 0 -> xyz=0.017 0 -0.000875 rpy=-1.5708 0 0
- joint rpf_joint: origin xyz=0.031 0 0.00245 rpy=0 0 1.17317577259539 -> xyz=0.031 0 0 rpy=0 0 1.17317577259539
- joint tca_joint: origin xyz=-0.024 0.014785 0.0072407 rpy=2.8032 -1.0121 1.9642 -> xyz=-0.024 0.01695 0.011491 rpy=2.8032 -1.0121 1.9642
- joint tcf_joint: origin xyz=-0.03245 -0.0217 0.055 rpy=0 0 0 -> xyz=-0.03245 -0.0217 0.0495 rpy=0 0 0
- joint tdf_joint: limit lower=-1.57 upper=1.57 effort=0 velocity=0 -> lower=0 upper=1.25 effort=0 velocity=0; origin xyz=0.025 0 0 rpy=0 0 0.128195437634862 -> xyz=0.025 0 0 rpy=0 0 0.1282
- joint tma_joint: origin xyz=0.025 0.00304267643461039 0.0026 rpy=-1.5707963267949 0.27478795531439 0 -> xyz=0.025 -0.0014573 0.0001 rpy=-1.5708 0.27479 0
- joint tmf_joint: origin xyz=0.0199999999999999 0.00199999999999999 -0.003 rpy=1.5707963267949 -0.346793637861002 0 -> xyz=0.02 0 0.0015 rpy=1.5708 -0.34679 0
