Commit message: V3 Consolidation
This reverts commit 2836796c89e944e73232c0c7851e8835ec383ce5.

File: src/hand_rviz/urdf/hand_urdf.urdf (robot description, URDF)
Before this commit: robot hand_rviz_urdf, 32 links, 31 joints
Links:
- removed link ids_link
- removed link mds_link
- removed link pds_link
- removed link rds_link
- removed link tds_link
- link hand_base_link: mass 1.41105557691145 -> 1.38812640347778
- link i_tip_link: mass 0.00010634 -> 9.6341391738565E-05
- link idf_link: mass 0.00334446738731233 -> 0.00213606646468497
- link ima_link: mass 0.00449002294753804 -> 0.00377097433248701
- link imf_link: mass 0.00428037699515229 -> 0.0035062778446748
- link ipf_link: mass 0.0017829399503603 -> 0.00108838501206663
- link m_tip_link: mass 0.00010634 -> 9.63413917385605E-05
- link mdf_link: mass 0.00334446743318713 -> 0.00213606647535568
- link mma_link: mass 0.00449001647184619 -> 0.00377096877435373
- link mmf_link: mass 0.00428037699020959 -> 0.0035062779381524
- link mpf_link: mass 0.00178293992081719 -> 0.00108838501206664
- link p_tip_link: mass 0.00010634 -> 9.63413917385593E-05
- link pdf_link: mass 0.00334446738731236 -> 0.00213606649935726
- link pma_link: mass 0.0044900248403291 -> 0.00377097300672915
- link pmf_link: mass 0.00428037700888134 -> 0.00350627798987508
- link ppf_link: mass 0.00178293983469879 -> 0.00108838501206663
- link r_tip_link: mass 0.00010634 -> 9.63413917385707E-05
- link rdf_link: mass 0.0033444674327742 -> 0.002136066487395
- link rma_link: mass 0.00449002148418832 -> 0.00377097155039619
- link rmf_link: mass 0.00428037699145368 -> 0.00350627800305113
- link rpf_link: mass 0.00178293986878615 -> 0.00108838501206664
- link t_tip_link: mass 0.000106342041717247 -> 9.63413917384506E-05
- link tca_link: mass 0.00511850580963509 -> 0.00499478923208696
- link tcf_link: mass 0.00505286263408417 -> 0.00484999590725353
- link tdf_link: mass 0.00311228154218926 -> 0.00217689228300246
- link tma_link: mass 0.00329743064165085 -> 0.00320272686969075
- link tmf_link: mass 0.00178293997137009 -> 0.000948811114997913
Joints:
- removed joint i_tip_joint
- removed joint ids_joint
- removed joint m_tip_joint
- removed joint mds_joint
- removed joint p_tip_joint
- removed joint pds_joint
- removed joint r_tip_joint
- removed joint rds_joint
- removed joint t_tip_joint
- removed joint tds_joint
- added joint i_tip: type fixed, parent idf_link, child i_tip_link, origin xyz=0.0091323 0 0 rpy=0 0 0, axis 0 0 0
- added joint m_tip: type fixed, parent mdf_link, child m_tip_link, origin xyz=0.0091323 0 0 rpy=0 0 0, axis 0 0 0
- added joint p_tip: type fixed, parent pdf_link, child p_tip_link, origin xyz=0.00913233682828257 0 0 rpy=0 0 0, axis 0 0 0
- added joint r_tip: type fixed, parent rdf_link, child r_tip_link, origin xyz=0.00913233682828257 0 0 rpy=0 0 0, axis 0 0 0
- added joint t_tip: type fixed, parent tdf_link, child t_tip_link, origin xyz=0.012137 0 0 rpy=0 0 0, axis 0 0 0
- joint idf_joint: limit lower=-0.175 upper=1.25 effort=0 velocity=0 -> lower=0 upper=1.25 effort=0 velocity=0; origin xyz=0.028 0 0 rpy=0 0 0.42403 -> xyz=0.02618 0 0 rpy=0 0 0.39762
- joint ima_joint: origin xyz=-0.030453 -0.042025 0.11347 rpy=1.5708 -1.4573 3.1416 -> xyz=-0.030085 -0.0405 0.11024 rpy=-1.5708 -1.4573 -3.1416
- joint imf_joint: origin xyz=0.017 0 0.0004 rpy=1.5708 0 0 -> xyz=0.017 0 -0.000875 rpy=-1.5708 0 0
- joint ipf_joint: limit lower=-0.650 upper=1.57 effort=0 velocity=0 -> lower=-0.873 upper=1.57 effort=0 velocity=0; origin xyz=0.032 0 0 rpy=0 0 1.1468 -> xyz=0.031 0 0 rpy=0 0 1.1732
- joint mdf_joint: limit lower=-0.175 upper=1.25 effort=0 velocity=0 -> lower=0 upper=1.25 effort=0 velocity=0; origin xyz=0.028 0 0 rpy=0 0 0.42403 -> xyz=0.02618 0 0 rpy=0 0 0.39762
- joint mma_joint: origin xyz=-0.010408 -0.042025 0.12371 rpy=1.5708 -1.5272 -3.1416 -> xyz=-0.010267 -0.0405 0.12046 rpy=-1.5708 -1.5272 -3.1416
- joint mmf_joint: origin xyz=0.017 0 0.0004 rpy=1.5708 0 0 -> xyz=0.017 0 -0.000875 rpy=-1.5708 0 0
- joint mpf_joint: limit lower=-0.650 upper=1.57 effort=0 velocity=0 -> lower=-0.873 upper=1.57 effort=0 velocity=0; origin xyz=0.032 0 0 rpy=0 0 1.1468 -> xyz=0.031 0 0 rpy=0 0 1.1732
- joint pdf_joint: limit lower=-0.175 upper=1.25 effort=0 velocity=0 -> lower=0 upper=1.25 effort=0 velocity=0; origin xyz=0.028 0 0 rpy=0 0 0.42403 -> xyz=0.02618 0 0 rpy=0 0 0.397620554199505
- joint pma_joint: origin xyz=0.030453 -0.042025 0.11347 rpy=-1.5708 -1.4573 0 -> xyz=0.030085 -0.0405 0.11024 rpy=1.5708 -1.4573 0
- joint pmf_joint: origin xyz=0.017 0 0.0004 rpy=1.5708 0 0 -> xyz=0.017 0 -0.000875 rpy=-1.5707963267949 0 0
- joint ppf_joint: limit lower=-0.650 upper=1.57 effort=0 velocity=0 -> lower=-0.873 upper=1.57 effort=0 velocity=0; origin xyz=0.032 0 0 rpy=0 0 1.1468 -> xyz=0.031 0 0 rpy=0 0 1.17317577259539
- joint rdf_joint: limit lower=-0.175 upper=1.25 effort=0 velocity=0 -> lower=0 upper=1.25 effort=0 velocity=0; origin xyz=0.028 0 0 rpy=0 0 0.42403 -> xyz=0.02618 0 0 rpy=0 0 0.397620554199504
- joint rma_joint: origin xyz=0.010408 -0.042025 0.12371 rpy=-1.5708 -1.5272 0 -> xyz=0.010267 -0.0405 0.12046 rpy=1.5708 -1.5272 0
- joint rmf_joint: origin xyz=0.017 0 0.0004 rpy=1.5708 0 0 -> xyz=0.017 0 -0.000875 rpy=-1.5708 0 0
- joint rpf_joint: limit lower=-0.650 upper=1.57 effort=0 velocity=0 -> lower=-0.873 upper=1.57 effort=0 velocity=0; origin xyz=0.032 0 0 rpy=0 0 1.1468 -> xyz=0.031 0 0 rpy=0 0 1.17317577259539
- joint tca_joint: origin xyz=-0.024 0.016626 0.011678 rpy=2.7701 -1.0044 2.0034 -> xyz=-0.024 0.01695 0.011491 rpy=2.8032 -1.0121 1.9642
- joint tcf_joint: origin xyz=-0.03305 -0.02155 0.0495 rpy=0 0 0 -> xyz=-0.03245 -0.0217 0.0495 rpy=0 0 0
- joint tdf_joint: limit lower=-0.175 upper=1.25 effort=0 velocity=0 -> lower=0 upper=1.25 effort=0 velocity=0; origin xyz=0.028 0 0 rpy=0 0 0.42403 -> xyz=0.025 0 0 rpy=0 0 0.1282
- joint tma_joint: origin xyz=0.025 0.000975 0.000475 rpy=-1.5708 0 0 -> xyz=0.025 -0.0014573 0.0001 rpy=-1.5708 0.27479 0
- joint tmf_joint: limit lower=-0.650 upper=1.57 effort=0 velocity=0 -> lower=-0.8 upper=1.57 effort=0 velocity=0; origin xyz=0.023 -0.000125 -0.003475 rpy=1.5708 -1.1468 0 -> xyz=0.02 0 0.0015 rpy=1.5708 -0.34679 0

File: src/hand_rviz/urdf/hand_urdf_cf.urdf (robot description, URDF)
Before this commit: robot hand_rviz_urdf, 32 links, 31 joints
Links:
- removed link ids_link
- removed link mds_link
- removed link pds_link
- removed link rds_link
- removed link tds_link
- link hand_base_link: mass 1.41105557691145 -> 1.38812640347778; geometry collision mesh filename=package://hand_rviz/urdf/meshes/hand_base_link.STL; visual mesh filename=package://hand_rviz/urdf/meshes/hand_base_link.STL
- link i_tip_link: mass 0.00010634 -> 9.6341391738565E-05; geometry collision mesh filename=package://hand_rviz/urdf/meshes/i_tip_link.STL; visual mesh filename=package://hand_rviz/urdf/meshes/i_tip_link.STL
- link idf_link: mass 0.00334446738731233 -> 0.00213606646468497; geometry collision mesh filename=package://hand_rviz/urdf/meshes/idf_link.STL; visual mesh filename=package://hand_rviz/urdf/meshes/idf_link.STL
- link ima_link: mass 0.00449002294753804 -> 0.00377097433248701; geometry collision mesh filename=package://hand_rviz/urdf/meshes/ima_link.STL; visual mesh filename=package://hand_rviz/urdf/meshes/ima_link.STL
- link imf_link: mass 0.00428037699515229 -> 0.0035062778446748; geometry collision mesh filename=package://hand_rviz/urdf/meshes/imf_link.STL; visual mesh filename=package://hand_rviz/urdf/meshes/imf_link.STL
- link ipf_link: mass 0.0017829399503603 -> 0.00108838501206663; geometry collision mesh filename=package://hand_rviz/urdf/meshes/ipf_link.STL; visual mesh filename=package://hand_rviz/urdf/meshes/ipf_link.STL
- link m_tip_link: mass 0.00010634 -> 9.63413917385605E-05; geometry collision mesh filename=package://hand_rviz/urdf/meshes/m_tip_link.STL; visual mesh filename=package://hand_rviz/urdf/meshes/m_tip_link.STL
- link mdf_link: mass 0.00334446743318713 -> 0.00213606647535568; geometry collision mesh filename=package://hand_rviz/urdf/meshes/mdf_link.STL; visual mesh filename=package://hand_rviz/urdf/meshes/mdf_link.STL
- link mma_link: mass 0.00449001647184619 -> 0.00377096877435373; geometry collision mesh filename=package://hand_rviz/urdf/meshes/mma_link.STL; visual mesh filename=package://hand_rviz/urdf/meshes/mma_link.STL
- link mmf_link: mass 0.00428037699020959 -> 0.0035062779381524; geometry collision mesh filename=package://hand_rviz/urdf/meshes/mmf_link.STL; visual mesh filename=package://hand_rviz/urdf/meshes/mmf_link.STL
- link mpf_link: mass 0.00178293992081719 -> 0.00108838501206664; geometry collision mesh filename=package://hand_rviz/urdf/meshes/mpf_link.STL; visual mesh filename=package://hand_rviz/urdf/meshes/mpf_link.STL
- link p_tip_link: mass 0.00010634 -> 9.63413917385593E-05; geometry collision mesh filename=package://hand_rviz/urdf/meshes/p_tip_link.STL; visual mesh filename=package://hand_rviz/urdf/meshes/p_tip_link.STL
- link pdf_link: mass 0.00334446738731236 -> 0.00213606649935726; geometry collision mesh filename=package://hand_rviz/urdf/meshes/pdf_link.STL; visual mesh filename=package://hand_rviz/urdf/meshes/pdf_link.STL
- link pma_link: mass 0.0044900248403291 -> 0.00377097300672915; geometry collision mesh filename=package://hand_rviz/urdf/meshes/pma_link.STL; visual mesh filename=package://hand_rviz/urdf/meshes/pma_link.STL
- link pmf_link: mass 0.00428037700888134 -> 0.00350627798987508; geometry collision mesh filename=package://hand_rviz/urdf/meshes/pmf_link.STL; visual mesh filename=package://hand_rviz/urdf/meshes/pmf_link.STL
- link ppf_link: mass 0.00178293983469879 -> 0.00108838501206663; geometry collision mesh filename=package://hand_rviz/urdf/meshes/ppf_link.STL; visual mesh filename=package://hand_rviz/urdf/meshes/ppf_link.STL
- link r_tip_link: mass 0.00010634 -> 9.63413917385707E-05; geometry collision mesh filename=package://hand_rviz/urdf/meshes/r_tip_link.STL; visual mesh filename=package://hand_rviz/urdf/meshes/r_tip_link.STL
- link rdf_link: mass 0.0033444674327742 -> 0.002136066487395; geometry collision mesh filename=package://hand_rviz/urdf/meshes/rdf_link.STL; visual mesh filename=package://hand_rviz/urdf/meshes/rdf_link.STL
- link rma_link: mass 0.00449002148418832 -> 0.00377097155039619; geometry collision mesh filename=package://hand_rviz/urdf/meshes/rma_link.STL; visual mesh filename=package://hand_rviz/urdf/meshes/rma_link.STL
- link rmf_link: mass 0.00428037699145368 -> 0.00350627800305113; geometry collision mesh filename=package://hand_rviz/urdf/meshes/rmf_link.STL; visual mesh filename=package://hand_rviz/urdf/meshes/rmf_link.STL
- link rpf_link: mass 0.00178293986878615 -> 0.00108838501206664; geometry collision mesh filename=package://hand_rviz/urdf/meshes/rpf_link.STL; visual mesh filename=package://hand_rviz/urdf/meshes/rpf_link.STL
- link t_tip_link: mass 0.000106342041717247 -> 9.63413917384506E-05; geometry collision mesh filename=package://hand_rviz/urdf/meshes/t_tip_link.STL; visual mesh filename=package://hand_rviz/urdf/meshes/t_tip_link.STL
- link tca_link: mass 0.00511850580963509 -> 0.00499478923208696; geometry collision mesh filename=package://hand_rviz/urdf/meshes/tca_link.STL; visual mesh filename=package://hand_rviz/urdf/meshes/tca_link.STL
- link tcf_link: mass 0.00505286263408417 -> 0.00484999590725353; geometry collision mesh filename=package://hand_rviz/urdf/meshes/tcf_link.STL; visual mesh filename=package://hand_rviz/urdf/meshes/tcf_link.STL
- link tdf_link: mass 0.00311228154218926 -> 0.00217689228300246; geometry collision mesh filename=package://hand_rviz/urdf/meshes/tdf_link.STL; visual mesh filename=package://hand_rviz/urdf/meshes/tdf_link.STL
- link tma_link: mass 0.00329743064165085 -> 0.00320272686969075; geometry collision mesh filename=package://hand_rviz/urdf/meshes/tma_link.STL; visual mesh filename=package://hand_rviz/urdf/meshes/tma_link.STL
- link tmf_link: mass 0.00178293997137009 -> 0.000948811114997913; geometry collision mesh filename=package://hand_rviz/urdf/meshes/tmf_link.STL; visual mesh filename=package://hand_rviz/urdf/meshes/tmf_link.STL
Joints:
- removed joint i_tip_joint
- removed joint ids_joint
- removed joint m_tip_joint
- removed joint mds_joint
- removed joint p_tip_joint
- removed joint pds_joint
- removed joint r_tip_joint
- removed joint rds_joint
- removed joint t_tip_joint
- removed joint tds_joint
- added joint i_tip: type fixed, parent idf_link, child i_tip_link, origin xyz=0.0091323 0 0 rpy=0 0 0, axis 0 0 0
- added joint m_tip: type fixed, parent mdf_link, child m_tip_link, origin xyz=0.0091323 0 0 rpy=0 0 0, axis 0 0 0
- added joint p_tip: type fixed, parent pdf_link, child p_tip_link, origin xyz=0.00913233682828257 0 0 rpy=0 0 0, axis 0 0 0
- added joint r_tip: type fixed, parent rdf_link, child r_tip_link, origin xyz=0.00913233682828257 0 0 rpy=0 0 0, axis 0 0 0
- added joint t_tip: type fixed, parent tdf_link, child t_tip_link, origin xyz=0.012137 0 0 rpy=0 0 0, axis 0 0 0
- joint idf_joint: limit lower=-0.175 upper=1.25 effort=0 velocity=0 -> lower=0 upper=1.25 effort=0 velocity=0; origin xyz=0.028 0 0 rpy=0 0 0.42403 -> xyz=0.02618 0 0 rpy=0 0 0.39762
- joint ima_joint: origin xyz=-0.030453 -0.042025 0.11347 rpy=1.5708 -1.4573 3.1416 -> xyz=-0.030085 -0.0405 0.11024 rpy=-1.5708 -1.4573 -3.1416
- joint imf_joint: origin xyz=0.017 0 0.0004 rpy=1.5708 0 0 -> xyz=0.017 0 -0.000875 rpy=-1.5708 0 0
- joint ipf_joint: origin xyz=0.032 0 0 rpy=0 0 1.1468 -> xyz=0.031 0 0 rpy=0 0 1.1732
- joint mdf_joint: limit lower=-0.175 upper=1.25 effort=0 velocity=0 -> lower=0 upper=1.25 effort=0 velocity=0; origin xyz=0.028 0 0 rpy=0 0 0.42403 -> xyz=0.02618 0 0 rpy=0 0 0.39762
- joint mma_joint: origin xyz=-0.010408 -0.042025 0.12371 rpy=1.5708 -1.5272 -3.1416 -> xyz=-0.010267 -0.0405 0.12046 rpy=-1.5708 -1.5272 -3.1416
- joint mmf_joint: origin xyz=0.017 0 0.0004 rpy=1.5708 0 0 -> xyz=0.017 0 -0.000875 rpy=-1.5708 0 0
- joint mpf_joint: origin xyz=0.032 0 0 rpy=0 0 1.1468 -> xyz=0.031 0 0 rpy=0 0 1.1732
- joint pdf_joint: limit lower=-0.175 upper=1.25 effort=0 velocity=0 -> lower=0 upper=1.25 effort=0 velocity=0; origin xyz=0.028 0 0 rpy=0 0 0.42403 -> xyz=0.02618 0 0 rpy=0 0 0.397620554199505
- joint pma_joint: origin xyz=0.030453 -0.042025 0.11347 rpy=-1.5708 -1.4573 0 -> xyz=0.030085 -0.0405 0.11024 rpy=1.5708 -1.4573 0
- joint pmf_joint: origin xyz=0.017 0 0.0004 rpy=1.5708 0 0 -> xyz=0.017 0 -0.000875 rpy=-1.5707963267949 0 0
- joint ppf_joint: origin xyz=0.032 0 0 rpy=0 0 1.1468 -> xyz=0.031 0 0 rpy=0 0 1.17317577259539
- joint rdf_joint: limit lower=-0.175 upper=1.25 effort=0 velocity=0 -> lower=0 upper=1.25 effort=0 velocity=0; origin xyz=0.028 0 0 rpy=0 0 0.42403 -> xyz=0.02618 0 0 rpy=0 0 0.397620554199504
- joint rma_joint: origin xyz=0.010408 -0.042025 0.12371 rpy=-1.5708 -1.5272 0 -> xyz=0.010267 -0.0405 0.12046 rpy=1.5708 -1.5272 0
- joint rmf_joint: origin xyz=0.017 0 0.0004 rpy=1.5708 0 0 -> xyz=0.017 0 -0.000875 rpy=-1.5708 0 0
- joint rpf_joint: origin xyz=0.032 0 0 rpy=0 0 1.1468 -> xyz=0.031 0 0 rpy=0 0 1.17317577259539
- joint tca_joint: origin xyz=-0.024 0.016626 0.011678 rpy=2.7701 -1.0044 2.0034 -> xyz=-0.024 0.01695 0.011491 rpy=2.8032 -1.0121 1.9642
- joint tcf_joint: origin xyz=-0.03305 -0.02155 0.0495 rpy=0 0 0 -> xyz=-0.03245 -0.0217 0.0495 rpy=0 0 0
- joint tdf_joint: limit lower=-0.175 upper=1.25 effort=0 velocity=0 -> lower=0 upper=1.25 effort=0 velocity=0; origin xyz=0.028 0 0 rpy=0 0 0.42403 -> xyz=0.025 0 0 rpy=0 0 0.1282
- joint tma_joint: origin xyz=0.025 0.000975 0.000475 rpy=-1.5708 0 0 -> xyz=0.025 -0.0014573 0.0001 rpy=-1.5708 0.27479 0
- joint tmf_joint: origin xyz=0.023 -0.000125 -0.003475 rpy=1.5708 -1.1468 0 -> xyz=0.02 0 0.0015 rpy=1.5708 -0.34679 0
